Commit message: diffdrive hardware, add gitignore, clean up

File: control_ws/src/diffdrive_gpio/description/urdf/diffbot.core.xacro (robot description, xacro)
@@ -1,5 +1,5 @@
 <?xml version="1.0"?>
 <robot xmlns:xacro="http://www.ros.org/wiki/xacro">
-    <xacro:include filename="inertial_macros.xacro"/>
+    <xacro:include filename="$(find diffdrive_gpio)/urdf/inertial_macros.xacro" />
     <!-- Updated Parameters based on provided robot specifications -->
     <xacro:property name="chassis_length" value="0.245"/>

File: robox_ws/src/robox/description/lidar_example.xacro (robot description, xacro)
@@ -4,10 +4,10 @@
         <parent link="chassis"/>
         <child link="laser_frame"/>
-        <origin xyz="0.122 0 0.145" rpy="0 0 0"/> <!-- Adjusted according to ground to LiDAR top: 14.5cm -->
+        <origin xyz="0.122 0 0.212" rpy="0 0 0"/>
     </joint>
     <link name="laser_frame">
         <visual>
             <geometry>
-                <cylinder radius="0.05" length="0.04"/>  <!-- Approximate size of LiDAR -->
+                <cylinder radius="0.05" length="0.04"/>
             </geometry>
             <material name="black"/>
@@ -25,6 +25,5 @@
             </geometry>
         </collision>
-        <!-- LiDAR inertial properties -->
-        <xacro:inertial_cylinder mass="0.125" length="0.04" radius="0.05"> <!-- Updated mass for LiDAR -->
+        <xacro:inertial_cylinder mass="0.1" length="0.04" radius="0.05">
             <origin xyz="0 0 0" rpy="0 0 0"/>
         </xacro:inertial_cylinder>

File: robox_ws/src/robox/description/robot_core_example.xacro (robot description, xacro)
@@ -1,21 +1,19 @@
 <?xml version="1.0"?>
-<robot xmlns:xacro="http://www.ros.org/wiki/xacro">
+<robot xmlns:xacro="http://www.ros.org/wiki/xacro" >
     <xacro:include filename="inertial_macros.xacro"/>
-    <!-- Updated Parameters based on provided robot specifications -->
-    <xacro:property name="chassis_length" value="0.245"/>
-    <xacro:property name="chassis_width" value="0.145"/>
-    <xacro:property name="chassis_height" value="0.075"/> <!-- Ground to robot top -->
-    <xacro:property name="chassis_mass" value="1.045"/> <!-- Updated chassis mass -->
-    <xacro:property name="wheel_radius" value="0.0325"/>  <!-- Wheel radius: half of 6.5cm diameter -->
-    <xacro:property name="wheel_thickness" value="0.0275"/> <!-- Wheel thickness 2.75cm -->
-    <xacro:property name="wheel_mass" value="0.06"/> <!-- Updated wheel mass for each wheel -->
-    <xacro:property name="wheel_offset_x" value="0.0975"/> <!-- Main wheels: 7.5cm from the back -->
-    <xacro:property name="wheel_offset_y" value="0.0725"/> <!-- Half of chassis_width (0.145/2) -->
+    <xacro:property name="chassis_length" value="0.335"/>
+    <xacro:property name="chassis_width" value="0.265"/>
+    <xacro:property name="chassis_height" value="0.138"/>
+    <xacro:property name="chassis_mass" value="1.0"/>
+    <xacro:property name="wheel_radius" value="0.033"/>
+    <xacro:property name="wheel_thickness" value="0.026"/>
+    <xacro:property name="wheel_mass" value="0.05"/>
+    <xacro:property name="wheel_offset_x" value="0.226"/>
+    <xacro:property name="wheel_offset_y" value="0.1485"/>
     <xacro:property name="wheel_offset_z" value="0.01"/>
-    <xacro:property name="caster_wheel_radius" value="0.005"/> <!-- Caster wheel radius: 1cm diameter -->
-    <xacro:property name="caster_wheel_mass" value="0.01"/> <!-- Very light caster wheel -->
-    <xacro:property name="caster_wheel_offset_x" value="0.03"/> <!-- Caster wheel: 3cm from the front -->
+    <xacro:property name="caster_wheel_radius" value="0.01"/>
+    <xacro:property name="caster_wheel_mass" value="0.01"/>
+    <xacro:property name="caster_wheel_offset_x" value="0.075"/>
     <xacro:property name="caster_wheel_offset_z" value="${wheel_offset_z - wheel_radius + caster_wheel_radius}"/>
-    <!-- Materials for visualization -->
     <material name="white">
         <color rgba="1 1 1 1" />
@@ -36,5 +34,5 @@
     <link name="base_link">
     </link>
-    <!-- BASE FOOTPRINT LINK -->
+    <!-- BASE_FOOTPRINT LINK -->
     <joint name="base_footprint_joint" type="fixed">
         <parent link="base_link"/>
@@ -64,9 +62,11 @@
             </geometry>
         </collision>
-        <!-- Updated chassis mass -->
-        <xacro:inertial_box mass="${chassis_mass}" x="${chassis_length}" y="${chassis_width}" z="${chassis_height}">
+        <xacro:inertial_box mass="0.5" x="${chassis_length}" y="${chassis_width}" z="${chassis_height}">
             <origin xyz="${chassis_length/2} 0 ${chassis_height/2}" rpy="0 0 0"/>
         </xacro:inertial_box>
     </link>
+    <gazebo reference="chassis">
+        <material>Gazebo/Orange</material>
+    </gazebo>
     <!-- LEFT WHEEL LINK -->
     <joint name="left_wheel_joint" type="continuous">
@@ -88,9 +88,11 @@
             </geometry>
         </collision>
-        <!-- Updated wheel mass -->
         <xacro:inertial_cylinder mass="${wheel_mass}" length="${wheel_thickness}" radius="${wheel_radius}">
             <origin xyz="0 0 0" rpy="0 0 0"/>
         </xacro:inertial_cylinder>
     </link>
+    <gazebo reference="left_wheel">
+        <material>Gazebo/Blue</material>
+    </gazebo>
     <!-- RIGHT WHEEL LINK -->
     <joint name="right_wheel_joint" type="continuous">
@@ -112,9 +114,11 @@
             </geometry>
         </collision>
-        <!-- Updated wheel mass -->
         <xacro:inertial_cylinder mass="${wheel_mass}" length="${wheel_thickness}" radius="${wheel_radius}">
             <origin xyz="0 0 0" rpy="0 0 0"/>
         </xacro:inertial_cylinder>
     </link>
+    <gazebo reference="right_wheel">
+        <material>Gazebo/Blue</material>
+    </gazebo>
     <!-- CASTER WHEEL LINK -->
     <joint name="caster_wheel_joint" type="fixed">
@@ -139,3 +143,8 @@
         </xacro:inertial_sphere>
     </link>
+    <gazebo reference="caster_wheel">
+        <material>Gazebo/White</material>
+        <mu1 value="0.001"/>
+        <mu2 value="0.001"/>
+    </gazebo>
 </robot>

File: robox_ws/src/robox/description/ros2_control.xacro (robot description, xacro)
@@ -1,31 +1,32 @@
 <?xml version="1.0"?>
 <robot xmlns:xacro="http://www.ros.org/wiki/xacro">
-    <ros2_control name="RealRobot" type="system">
-        <hardware>
-            <plugin>diffdrive_arduino/DiffDriveArduino</plugin>
-            <param name="left_wheel_name">left_wheel_joint</param>
-            <param name="right_wheel_name">right_wheel_joint</param>
-            <!-- <param name="loop_rate">30</param> -->
-            <!-- <param name="device">/dev/ttyUSB0</param>
-            <param name="baud_rate">57600</param> -->
-            <param name="timeout">1000</param>
-            <param name="enc_counts_per_rev">680</param>
-        </hardware>
-        <joint name="left_wheel_joint">
-            <command_interface name="velocity">
-                <param name="min">-10</param>
-                <param name="max">10</param>
-            </command_interface>
-            <state_interface name="velocity"/>
-            <state_interface name="position"/>
-        </joint>
-        <joint name="right_wheel_joint">
-            <command_interface name="velocity">
-                <param name="min">-10</param>
-                <param name="max">10</param>
-            </command_interface>
-            <state_interface name="velocity"/>
-            <state_interface name="position"/>
-        </joint>
-    </ros2_control>
+  <ros2_control name="diffbot_control" type="system">
+    <hardware>
+      <plugin>diffdrive_gpio/DiffDriveGPIOHardware</plugin>
+      <!-- Hardware configuration parameters for GPIO -->
+      <param name="left_wheel_name">left_wheel_joint</param>
+      <param name="right_wheel_name">right_wheel_joint</param>
+      <!-- GPIO pin numbers for both encoder channels and motors -->
+      <param name="gpio_left_encoder_a">5</param>   <!-- GPIO pin for left encoder (Channel A) -->
+      <param name="gpio_left_encoder_b">6</param>   <!-- GPIO pin for left encoder (Channel B) -->
+      <param name="gpio_right_encoder_a">20</param> <!-- GPIO pin for right encoder (Channel A) -->
+      <param name="gpio_right_encoder_b">21</param> <!-- GPIO pin for right encoder (Channel B) -->
+      <param name="gpio_left_motor">22</param>      <!-- GPIO pin for left motor -->
+      <param name="gpio_right_motor">23</param>     <!-- GPIO pin for right motor -->
+      <!-- Other configuration parameters -->
+      <param name="loop_rate">50.0</param>        <!-- Control loop rate in Hz -->
+      <param name="enc_counts_per_rev">660</param> <!-- Encoder counts per revolution -->
+    </hardware>
+    <!-- Joint definitions for left and right wheels -->
+    <joint name="left_wheel_joint">
+      <command_interface name="velocity"/>
+      <state_interface name="position"/>
+      <state_interface name="velocity"/>
+    </joint>
+    <joint name="right_wheel_joint">
+      <command_interface name="velocity"/>
+      <state_interface name="position"/>
+      <state_interface name="velocity"/>
+    </joint>
+  </ros2_control>
 </robot>
