Commit message: arduino diffdrive

File: control_ws/src/diffdrive_arduino/description/urdf/diffbot.core.xacro (robot description, xacro)
@@ -1,16 +1,16 @@
 <?xml version="1.0"?>
 <robot xmlns:xacro="http://www.ros.org/wiki/xacro">
-    <xacro:include filename="inertial_macros.xacro"/>
+    <xacro:include filename="$(find diffdrive_arduino)/urdf/inertial_macros.xacro" />
     <!-- Updated Parameters based on provided robot specifications -->
-    <xacro:property name="chassis_length" value="0.245"/> <!-- Body length 24.5cm -->
-    <xacro:property name="chassis_width" value="0.145"/> <!-- Body width 14.5cm -->
+    <xacro:property name="chassis_length" value="0.245"/>
+    <xacro:property name="chassis_width" value="0.145"/>
     <xacro:property name="chassis_height" value="0.075"/> <!-- Ground to robot top -->
-    <xacro:property name="chassis_mass" value="1.3"/> <!-- Updated chassis mass -->
-    <xacro:property name="wheel_radius" value="0.035"/>  <!-- Wheel radius: half of 7cm diameter -->
-    <xacro:property name="wheel_thickness" value="0.027"/> <!-- Wheel thickness 2.7cm -->
+    <xacro:property name="chassis_mass" value="1.045"/> <!-- Updated chassis mass -->
+    <xacro:property name="wheel_radius" value="0.0325"/>  <!-- Wheel radius: half of 6.5cm diameter -->
+    <xacro:property name="wheel_thickness" value="0.0275"/> <!-- Wheel thickness 2.75cm -->
     <xacro:property name="wheel_mass" value="0.06"/> <!-- Updated wheel mass for each wheel -->
-    <xacro:property name="wheel_offset_x" value="${chassis_length - 0.08}"/> <!-- Main wheels: 8cm from the front -->
-    <xacro:property name="wheel_offset_y" value="${chassis_width/2 + wheel_thickness}"/> <!-- Half of chassis_width (0.145/2) -->
-    <xacro:property name="wheel_offset_z" value="${wheel_radius - caster_wheel_radius}"/>
+    <xacro:property name="wheel_offset_x" value="0.0975"/> <!-- Main wheels: 7.5cm from the back -->
+    <xacro:property name="wheel_offset_y" value="0.0725"/> <!-- Half of chassis_width (0.145/2) -->
+    <xacro:property name="wheel_offset_z" value="0.01"/>
     <xacro:property name="caster_wheel_radius" value="0.005"/> <!-- Caster wheel radius: 1cm diameter -->
     <xacro:property name="caster_wheel_mass" value="0.01"/> <!-- Very light caster wheel -->

File: robox_ws/src/robox/description/lidar.xacro (robot description, xacro)
@@ -4,10 +4,10 @@
         <parent link="chassis"/>
         <child link="laser_frame"/>
-        <origin xyz="0.122 0 0.145" rpy="0 0 0"/> <!-- Adjusted according to ground to LiDAR top: 14.5cm -->
+        <origin xyz="0.185 0 0.12" rpy="0 0 0"/> <!-- Adjusted according to ground to LiDAR top: 14.5cm -->
     </joint>
     <link name="laser_frame">
         <visual>
             <geometry>
-                <cylinder radius="0.05" length="0.04"/>  <!-- Approximate size of LiDAR -->
+                <cylinder radius="0.04" length="0.03"/>  <!-- Approximate size of LiDAR -->
             </geometry>
             <material name="black"/>
@@ -22,9 +22,8 @@
         <collision>
             <geometry>
-                <cylinder radius="0.05" length="0.04"/>
+                <cylinder radius="0.04" length="0.04"/>
             </geometry>
         </collision>
-        <!-- LiDAR inertial properties -->
-        <xacro:inertial_cylinder mass="0.125" length="0.04" radius="0.05"> <!-- Updated mass for LiDAR -->
+        <xacro:inertial_cylinder mass="0.125" length="0.04" radius="0.04"> <!-- Updated mass for LiDAR -->
             <origin xyz="0 0 0" rpy="0 0 0"/>
         </xacro:inertial_cylinder>

File: robox_ws/src/robox/description/robox.urdf.xacro (robot description, xacro)
@@ -1,4 +1,5 @@
 <?xml version="1.0"?>
-<robot xmlns:xacro="http://www.ros.org/wiki/xacro"  name="robox">
+<robot xmlns:xacro="http://www.ros.org/wiki/xacro" name="robox">
+    <xacro:include filename="ros2_control.xacro" />
     <xacro:include filename="robot_core.xacro" />
     <xacro:include filename="lidar.xacro" />

File: robox_ws/src/robox/description/ros2_control.xacro (robot description, xacro)
@@ -1,22 +1,20 @@
 <?xml version="1.0"?>
 <robot xmlns:xacro="http://www.ros.org/wiki/xacro">
-  <ros2_control name="diffbot_control" type="system">
+  <ros2_control name="diffbot_ros2_control" type="system">
     <hardware>
-      <plugin>diffdrive_gpio/DiffDriveGPIOHardware</plugin>
-      <!-- Hardware configuration parameters for GPIO -->
-      <param name="left_wheel_name">left_wheel_joint</param>
-      <param name="right_wheel_name">right_wheel_joint</param>
-      <!-- GPIO pin numbers for both encoder channels and motors -->
-      <param name="gpio_left_encoder_a">5</param>   <!-- GPIO pin for left encoder (Channel A) -->
-      <param name="gpio_left_encoder_b">6</param>   <!-- GPIO pin for left encoder (Channel B) -->
-      <param name="gpio_right_encoder_a">20</param> <!-- GPIO pin for right encoder (Channel A) -->
-      <param name="gpio_right_encoder_b">21</param> <!-- GPIO pin for right encoder (Channel B) -->
-      <param name="gpio_left_motor">22</param>      <!-- GPIO pin for left motor -->
-      <param name="gpio_right_motor">23</param>     <!-- GPIO pin for right motor -->
-      <!-- Other configuration parameters -->
-      <param name="loop_rate">50.0</param>        <!-- Control loop rate in Hz -->
-      <param name="enc_counts_per_rev">660</param> <!-- Encoder counts per revolution -->
+      <plugin>diffdrive_arduino/DiffDriveArduinoHardware</plugin>
+       <param name="left_wheel_name">left_wheel_joint</param>
+        <param name="right_wheel_name">right_wheel_joint</param>
+        <param name="loop_rate">30</param>
+        <!-- <param name="device">/dev/serial/by-path/platform-fd500000.pcie-pci-0000:01:00.0-usb-0:1.4:1.0-port0</param>       -->
+        <param name="device">/dev/ttyACM0</param>
+        <param name="baud_rate">57600</param>
+        <param name="timeout_ms">1000</param>
+        <param name="enc_counts_per_rev">330</param>
+        <param name="pid_p">20</param>
+        <param name="pid_d">12</param>
+        <param name="pid_i">0</param>
+        <param name="pid_o">50</param>
     </hardware>
-    <!-- Joint definitions for left and right wheels -->
     <joint name="left_wheel_joint">
       <command_interface name="velocity"/>
